Commit message: Add real robot control and hand-eye calibration workflows

File: sim_ws/validation/lidar_arm_blind/model.urdf (robot description, URDF)
Before this commit: robot mobile_dual_nero, 51 links, 50 joints
Links:
- added link upper_body_lift_rail, mass 4; collision box size=.06 .14 .86; visual box size=.06 .14 .86
Joints:
- removed joint dual_nero_mount_joint
- added joint upper_body_lift_joint: type prismatic, parent arm_mount_plate, child dual_nero_base_link, origin xyz=0 0 .006 rpy=0 0 0, axis 0 0 1, limit lower=0 upper=0.8 effort=2500 velocity=0.05
- added joint upper_body_lift_rail_mount: type fixed, parent arm_mount_plate, child upper_body_lift_rail, origin xyz=0 0 .006
